File: controller.kicad_pcb (KiCad board)
At the start: 2 copper layers, 147 x 80 mm, 94 parts, among them J1 1Wire, J2 VoltLink_target, J3 i2C, J4 OUTPUT, J5 OUTPUT, J6 AC IN, SW1 USER, U1 ESP32-WROOM-32D, U10 BC3223, U11 BC3223, U12 BC3223, U2 AMS1117-3.3, U3 BC3223, U4 BC3223, U5 BC3223, U6 BC3223, U7 BC3223, U8 BC3223, U9 BC3223

Commit message: revB release
Parts:
- removed the C7 at (139.0, 88.0)
- removed the D1 at (117.8, 72.8)
- removed the D2 at (97.0, 109.2)
- removed the PS1 at (93.0, 82.0) (x2)
- removed the R5 at (97.0, 106.0)
- removed U12: BC3223, voltlog:DIP-7_W7.62mm
- added FL1: EMI_Filter_LL, voltlog:UU9_choke, F.Cu at (68.5, 76.8)
- added N1: Housing, voltlog:BRT-80005, F.Cu at (111.0, 71.5)
- added PS1: HLK-PM03, Converter_ACDC:Converter_ACDC_HiLink_HLK-PMxx, F.Cu at (80.2, 78.2)
- added TP2: IO12, TestPoint:TestPoint_Pad_D1.5mm, F.Cu at (135.0, 90.8)
- added TP3: IO34, TestPoint:TestPoint_Pad_D1.5mm, F.Cu at (140.0, 90.8)
- added TP4: IO35, TestPoint:TestPoint_Pad_D1.5mm, F.Cu at (137.5, 90.8)
- added TP5: 3V3, TestPoint:TestPoint_Pad_D1.5mm, F.Cu at (114.5, 89.5)
- C4: renamed from C3; footprint Capacitor_SMD:CP_Elec_10x10 -> Capacitor_SMD:CP_Elec_8x10.5
- F1: value 0.25A 250VAC -> 0.5A 250VAC
- J1: footprint Voltlog:KF235-5.0-3P -> Connector_PinHeader_2.54mm:PinHeader_1x03_P2.54mm_Vertical
- J4, J5: footprint Voltlog:KF235-5.0-10P -> TerminalBlock_RND:TerminalBlock_RND_205-00020_1x10_P5.00mm_Horizontal
- J6: footprint Voltlog:KF235-5.0-2P -> TerminalBlock_RND:TerminalBlock_RND_205-00012_1x02_P5.00mm_Horizontal
- R10, R11, R12, R13, R14, R15, R16, R17, R18, R9: footprint Resistor_THT:R_Axial_DIN0207_L6.3mm_D2.5mm_P10.16mm_Horizontal -> Resistor_THT:R_Axial_DIN0309_L9.0mm_D3.2mm_P5.08mm_Vertical
- R2: renamed from R19; value 1M -> 680K; footprint Resistor_THT:R_Axial_DIN0207_L6.3mm_D2.5mm_P10.16mm_Horizontal -> Resistor_THT:R_Axial_DIN0309_L9.0mm_D3.2mm_P12.70mm_Horizontal
- R8: value 330R -> 100R
- RN1, RN2, RN3: value 150R -> 75R
- RN4, RN5, RN6: value 470R -> 100R
- SW1: footprint Button_Switch_SMD:SW_SPST_PTS645 -> Button_Switch_THT:SW_Tactile_SKHH_Angled
- TP1: value 5V -> IO5; footprint TestPoint:TestPoint_Pad_D1.0mm -> TestPoint:TestPoint_Pad_D1.5mm
- U10, U11, U3, U4, U5, U6, U7, U8, U9: value BC3223 -> BC2213A; footprint voltlog:DIP-7_W7.62mm -> voltlog:SOIC-7
- U2: value AMS1117-3.3 -> BC2213A; footprint Package_TO_SOT_SMD:SOT-223-3_TabPin2 -> voltlog:SOIC-7
- moved U2 78.5 mm to (61.0, 61.0), turned to 0 degrees
- moved C7 39.9 mm to (105.8, 101.8), turned to 270 degrees
- moved SW1 38.9 mm to (108.8, 108.8), turned to 180 degrees
- moved R5 30.6 mm to (107.2, 101.8), turned to 90 degrees
- moved J4 22.7 mm to (117.0, 36.5)
- moved J5 21.2 mm to (167.0, 36.5)
- moved TP1 19.0 mm to (132.5, 90.8)
- moved U3 17.6 mm to (74.0, 61.0), turned to 0 degrees
- moved U4 17.6 mm to (87.0, 61.0), turned to 0 degrees
- moved U5 17.6 mm to (100.0, 61.0), turned to 0 degrees
- moved U6 17.6 mm to (113.0, 61.0), turned to 0 degrees
- moved U7 17.6 mm to (126.0, 61.0), turned to 0 degrees
- moved U11 17.1 mm to (178.0, 61.0), turned to 0 degrees
- moved U8 17.1 mm to (139.0, 61.0), turned to 0 degrees
- moved U9 17.1 mm to (152.0, 61.0), turned to 0 degrees
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- renumbered C11 to C10, C12 to C11, C13 to C12, C14 to C13, C15 to C14, C16 to C15, C17 to C16, C18 to C17, C19 to C18, C4 to C2, C2 to C3, C8 to C7, C9 to C8, C10 to C9, D3 to D1, D12 to D10, D13 to D11, D14 to D12, D4 to D2, D5 to D3, D6 to D4, D7 to D5, D8 to D6, D9 to D7, D10 to D8, D11 to D9, J3 to J2, J2 to J3, R2 to R3, R3 to R4, R4 to R5
Connections:
- C10 pad 1: Net-(C11-Pad1) -> Net-(C10-Pad1)
- C11 pad 1: Net-(C12-Pad1) -> Net-(C11-Pad1)
- C12 pad 1: Net-(C13-Pad1) -> Net-(C12-Pad1)
- C13 pad 1: Net-(C14-Pad1) -> Net-(C13-Pad1)
- C14 pad 1: Net-(C15-Pad1) -> Net-(C14-Pad1)
- C15 pad 1: Net-(C16-Pad1) -> Net-(C15-Pad1)
- C16 pad 1: Net-(C17-Pad1) -> Net-(C16-Pad1)
- C17 pad 1: Net-(C18-Pad1) -> Net-(C17-Pad1)
- C18 pad 1: Net-(C19-Pad1) -> Net-(C18-Pad1)
- C3 pad 1: +5V -> +3V3
- C4 pad 1: +5V -> +3V3
- C9 pad 1: Net-(C10-Pad1) -> Net-(C9-Pad1)
- D6 pad 2: /IO17 -> /IO15
- D7 pad 2: /IO16 -> /IO13
- D8 pad 2: /IO13 -> /IO14
- R10 pad 1: Net-(J4-Pad8) -> Net-(C10-Pad1)
- R10 pad 2: Net-(C11-Pad1) -> Net-(J4-Pad8)
- R11 pad 1: Net-(J4-Pad6) -> Net-(C11-Pad1)
- R11 pad 2: Net-(C12-Pad1) -> Net-(J4-Pad6)
- R12 pad 1: Net-(J4-Pad4) -> Net-(C12-Pad1)
- R12 pad 2: Net-(C13-Pad1) -> Net-(J4-Pad4)
- R13 pad 1: Net-(J4-Pad2) -> Net-(C13-Pad1)
- R13 pad 2: Net-(C14-Pad1) -> Net-(J4-Pad2)
- R14 pad 1: Net-(J5-Pad10) -> Net-(C14-Pad1)
- R14 pad 2: Net-(C15-Pad1) -> Net-(J5-Pad10)
- R15 pad 1: Net-(J5-Pad8) -> Net-(C15-Pad1)
- R15 pad 2: Net-(C16-Pad1) -> Net-(J5-Pad8)
- R16 pad 1: Net-(J5-Pad6) -> Net-(C16-Pad1)
- R16 pad 2: Net-(C17-Pad1) -> Net-(J5-Pad6)
- R17 pad 1: Net-(J5-Pad4) -> Net-(C17-Pad1)
- R17 pad 2: Net-(C18-Pad1) -> Net-(J5-Pad4)
- R18 pad 1: Net-(J5-Pad2) -> Net-(C18-Pad1)
- R18 pad 2: Net-(C19-Pad1) -> Net-(J5-Pad2)
- R9 pad 1: Net-(J4-Pad10) -> Net-(C9-Pad1)
- R9 pad 2: Net-(C10-Pad1) -> Net-(J4-Pad10)
- RN1 pad 4: /IO17 -> /IO15
- RN2 pad 1: /IO16 -> /IO13
- RN2 pad 2: /IO13 -> /IO14
- TP1 pad 1: +5V -> Net-(TP1-Pad1)
- U1 pad 13: Net-(U1-Pad13) -> /IO14
- U1 pad 23: Net-(U1-Pad23) -> /IO15
- U1 pad 27: /IO16 -> Net-(U1-Pad27)
- U1 pad 28: /IO17 -> Net-(U1-Pad28)
- U1 pad 29: Net-(U1-Pad29) -> Net-(TP1-Pad1)
- U10 pad 2: Net-(RN2-Pad5) -> Net-(RN3-Pad8)
- U10 pad 7: Net-(J5-Pad6) -> Net-(J5-Pad4)
- U11 pad 2: Net-(RN3-Pad8) -> Net-(RN3-Pad7)
- U11 pad 7: Net-(J5-Pad4) -> Net-(J5-Pad2)
- U2 pad 2: +3V3 -> Net-(RN1-Pad8)
- U2 pad 3: +5V -> GND
- U3 pad 2: Net-(RN1-Pad8) -> Net-(RN1-Pad7)
- U3 pad 7: Net-(J4-Pad10) -> Net-(J4-Pad8)
- U4 pad 2: Net-(RN1-Pad7) -> Net-(RN1-Pad6)
- U4 pad 7: Net-(J4-Pad8) -> Net-(J4-Pad6)
- U5 pad 2: Net-(RN1-Pad6) -> Net-(RN1-Pad5)
- U5 pad 7: Net-(J4-Pad6) -> Net-(J4-Pad4)
- U6 pad 2: Net-(RN1-Pad5) -> Net-(RN2-Pad8)
- U6 pad 7: Net-(J4-Pad4) -> Net-(J4-Pad2)
- U7 pad 2: Net-(RN2-Pad8) -> Net-(RN2-Pad7)
- U7 pad 7: Net-(J4-Pad2) -> Net-(J5-Pad10)
- U8 pad 2: Net-(RN2-Pad7) -> Net-(RN2-Pad6)
- U8 pad 7: Net-(J5-Pad10) -> Net-(J5-Pad8)
- U9 pad 2: Net-(RN2-Pad6) -> Net-(RN2-Pad5)
- U9 pad 7: Net-(J5-Pad8) -> Net-(J5-Pad6)
Routing:
- net GND: track 242.1 -> 160.6 mm, vias 98 -> 88
- net /Relay/F2_LIVE: track 263.0 -> 331.0 mm
- net Net-(TP3-Pad1): track 0.00 -> 64.6 mm, vias 0 -> 2
- net Net-(TP4-Pad1): track 0.00 -> 64.2 mm, vias 0 -> 2
- net Net-(TP2-Pad1): track 0.00 -> 51.5 mm, vias 0 -> 2
- net /NEUTRAL: track 313.5 -> 264.9 mm
- net +5V: track 40.8 -> 0.00 mm
- net Net-(TP1-Pad1): track 0.00 -> 33.9 mm, vias 0 -> 2
- net /IO14: track 0.00 -> 32.6 mm
- net /IO33: track 63.3 -> 88.5 mm, vias 2 -> 4
- net +3V3: track 146.2 -> 169.3 mm, vias 39 -> 15
- net /IO17: track 21.5 -> 0.00 mm
- net /IO16: track 20.7 -> 0.00 mm
- net Net-(FL1-Pad2): track 0.00 -> 19.9 mm
- net /IO15: track 0.00 -> 19.1 mm
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- removed copper zone on F.Cu, net +5V
Other:
- outline, holes or cut-outs redrawn
- board text added: "4521"
- board text added: "I2C"
- board text added: "IO12"
- board text added: "IO34"
- board text added: "IO35"
- board text added: "IO5"
- board text added: "revB"
- board text removed: "5V"
- board text removed: "Warning: revA has PS1 footprint mirrored!"
