File: controller.kicad_pcb (KiCad board)
At the start: 2 copper layers, 147 x 80 mm, 94 parts, among them J1 1Wire, J2 VoltLink_target, J3 i2C, J4 OUTPUT, J5 OUTPUT, J6 AC IN, SW1 USER, U1 ESP32-WROOM-32D, U10 BC3223, U11 BC3223, U12 BC3223, U2 AMS1117-3.3, U3 BC3223, U4 BC3223, U5 BC3223, U6 BC3223, U7 BC3223, U8 BC3223, U9 BC3223

Commit message: RevC initial release
Parts:
- removed the C7 at (139.0, 88.0)
- removed the D1 at (117.8, 72.8)
- removed the D2 at (97.0, 109.2)
- removed the PS1 at (93.0, 82.0) (x2)
- removed the R5 at (97.0, 106.0)
- removed U12: BC3223, voltlog:DIP-7_W7.62mm
- added FL1: EMI_Filter_LL, voltlog:UU9_choke, F.Cu at (68.5, 76.8)
- added N1: Housing, voltlog:BRT-80005, F.Cu at (111.0, 71.5)
- added PS1: HLK-PM03, Converter_ACDC:Converter_ACDC_HiLink_HLK-PMxx, F.Cu at (80.2, 78.2)
- added TP2: IO12, TestPoint:TestPoint_Pad_D1.5mm, F.Cu at (135.0, 90.8)
- added TP3: IO34, TestPoint:TestPoint_Pad_D1.5mm, F.Cu at (140.0, 90.8)
- added TP4: IO35, TestPoint:TestPoint_Pad_D1.5mm, F.Cu at (137.5, 90.8)
- added TP5: 3V3, TestPoint:TestPoint_Pad_D1.5mm, F.Cu at (114.5, 89.5)
- C4: renamed from C3; value 470uF -> 220uF; footprint Capacitor_SMD:CP_Elec_10x10 -> Capacitor_SMD:CP_Elec_8x10.5
- F1: value 0.25A 250VAC -> 0.5A 250VAC
- J1: footprint Voltlog:KF235-5.0-3P -> Connector_PinHeader_2.54mm:PinHeader_1x03_P2.54mm_Vertical
- J4, J5: footprint Voltlog:KF235-5.0-10P -> TerminalBlock_RND:TerminalBlock_RND_205-00020_1x10_P5.00mm_Horizontal
- J6: footprint Voltlog:KF235-5.0-2P -> TerminalBlock_RND:TerminalBlock_RND_205-00012_1x02_P5.00mm_Horizontal
- R10, R11, R12, R13, R14, R15, R16, R17, R18, R9: footprint Resistor_THT:R_Axial_DIN0207_L6.3mm_D2.5mm_P10.16mm_Horizontal -> Resistor_THT:R_Axial_DIN0309_L9.0mm_D3.2mm_P5.08mm_Vertical
- R2: renamed from R19; value 1M -> 680K; footprint Resistor_THT:R_Axial_DIN0207_L6.3mm_D2.5mm_P10.16mm_Horizontal -> Resistor_THT:R_Axial_DIN0309_L9.0mm_D3.2mm_P12.70mm_Horizontal
- R8: value 330R -> 100R
- RN1, RN2, RN3: value 150R -> 100R
- RN4, RN5, RN6: value 470R -> 100R
- RV1: value 10D471K -> 10D561K
- SW1: footprint Button_Switch_SMD:SW_SPST_PTS645 -> Button_Switch_THT:SW_Tactile_SKHH_Angled
- TP1: value 5V -> IO5; footprint TestPoint:TestPoint_Pad_D1.0mm -> TestPoint:TestPoint_Pad_D1.5mm
- U10, U11, U3, U4, U5, U6, U7, U8, U9: value BC3223 -> BC2213A; footprint voltlog:DIP-7_W7.62mm -> voltlog:SOIC-7
- U2: value AMS1117-3.3 -> BC2213A; footprint Package_TO_SOT_SMD:SOT-223-3_TabPin2 -> voltlog:SOIC-7
- moved U2 78.5 mm to (61.0, 61.0), turned to 0 degrees
- moved C7 39.9 mm to (105.8, 101.8), turned to 270 degrees
- moved SW1 38.9 mm to (108.8, 108.8), turned to 180 degrees
- moved R5 30.6 mm to (107.2, 101.8), turned to 90 degrees
- moved J4 22.7 mm to (117.0, 36.5)
- moved J5 21.2 mm to (167.0, 36.5)
- moved TP1 19.0 mm to (132.5, 90.8)
- moved U3 17.6 mm to (74.0, 61.0), turned to 0 degrees
- moved U4 17.6 mm to (87.0, 61.0), turned to 0 degrees
- moved U5 17.6 mm to (100.0, 61.0), turned to 0 degrees
- moved U6 17.6 mm to (113.0, 61.0), turned to 0 degrees
- moved U7 17.6 mm to (126.0, 61.0), turned to 0 degrees
- moved U11 17.1 mm to (178.0, 61.0), turned to 0 degrees
- moved U8 17.1 mm to (139.0, 61.0), turned to 0 degrees
- moved U9 17.1 mm to (152.0, 61.0), turned to 0 degrees
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- renumbered C11 to C10, C12 to C11, C13 to C12, C14 to C13, C15 to C14, C16 to C15, C17 to C16, C18 to C17, C19 to C18, C4 to C2, C2 to C3, C8 to C7, C9 to C8, C10 to C9, D3 to D1, D12 to D10, D13 to D11, D14 to D12, D4 to D2, D5 to D3, D6 to D4, D7 to D5, D8 to D6, D9 to D7, D10 to D8, D11 to D9, J3 to J2, J2 to J3, R2 to R3, R3 to R4, R4 to R5
Connections:
- C10 pad 1: Net-(C11-Pad1) -> Net-(C10-Pad1)
- C11 pad 1: Net-(C12-Pad1) -> Net-(C11-Pad1)
- C12 pad 1: Net-(C13-Pad1) -> Net-(C12-Pad1)
- C13 pad 1: Net-(C14-Pad1) -> Net-(C13-Pad1)
- C14 pad 1: Net-(C15-Pad1) -> Net-(C14-Pad1)
- C15 pad 1: Net-(C16-Pad1) -> Net-(C15-Pad1)
- C16 pad 1: Net-(C17-Pad1) -> Net-(C16-Pad1)
- C17 pad 1: Net-(C18-Pad1) -> Net-(C17-Pad1)
- C18 pad 1: Net-(C19-Pad1) -> Net-(C18-Pad1)
- C3 pad 1: +5V -> +3V3
- C4 pad 1: +5V -> +3V3
- C9 pad 1: Net-(C10-Pad1) -> Net-(C9-Pad1)
- D10 pad 1: Net-(D12-Pad1) -> Net-(D10-Pad1)
- D11 pad 1: Net-(D13-Pad1) -> Net-(D11-Pad1)
- D12 pad 1: Net-(D14-Pad1) -> Net-(D12-Pad1)
- D6 pad 2: /IO17 -> /IO15
- D7 pad 1: Net-(D9-Pad1) -> Net-(D7-Pad1)
- D7 pad 2: /IO16 -> /IO13
- D8 pad 1: Net-(D10-Pad1) -> Net-(D8-Pad1)
- D8 pad 2: /IO13 -> /IO14
- D9 pad 1: Net-(D11-Pad1) -> Net-(D9-Pad1)
- R10 pad 1: Net-(J4-Pad8) -> Net-(C10-Pad1)
- R10 pad 2: Net-(C11-Pad1) -> Net-(J4-Pad8)
- R11 pad 1: Net-(J4-Pad6) -> Net-(C11-Pad1)
- R11 pad 2: Net-(C12-Pad1) -> Net-(J4-Pad6)
- R12 pad 1: Net-(J4-Pad4) -> Net-(C12-Pad1)
- R12 pad 2: Net-(C13-Pad1) -> Net-(J4-Pad4)
- R13 pad 1: Net-(J4-Pad2) -> Net-(C13-Pad1)
- R13 pad 2: Net-(C14-Pad1) -> Net-(J4-Pad2)
- R14 pad 1: Net-(J5-Pad10) -> Net-(C14-Pad1)
- R14 pad 2: Net-(C15-Pad1) -> Net-(J5-Pad10)
- R15 pad 1: Net-(J5-Pad8) -> Net-(C15-Pad1)
- R15 pad 2: Net-(C16-Pad1) -> Net-(J5-Pad8)
- R16 pad 1: Net-(J5-Pad6) -> Net-(C16-Pad1)
- R16 pad 2: Net-(C17-Pad1) -> Net-(J5-Pad6)
- R17 pad 1: Net-(J5-Pad4) -> Net-(C17-Pad1)
- R17 pad 2: Net-(C18-Pad1) -> Net-(J5-Pad4)
- R18 pad 1: Net-(J5-Pad2) -> Net-(C18-Pad1)
- R18 pad 2: Net-(C19-Pad1) -> Net-(J5-Pad2)
- R9 pad 1: Net-(J4-Pad10) -> Net-(C9-Pad1)
- R9 pad 2: Net-(C10-Pad1) -> Net-(J4-Pad10)
- RN1 pad 4: /IO17 -> (no net)
- RN1 pad 5: Net-(RN1-Pad5) -> (no net)
- RN2 pad 1: /IO16 -> (no net)
- RN2 pad 2: /IO13 -> /IO15
- RN2 pad 3: /IO27 -> /IO13
- RN2 pad 4: /IO26 -> (no net)
- RN2 pad 5: Net-(RN2-Pad5) -> (no net)
- RN2 pad 8: Net-(RN2-Pad8) -> (no net)
- RN3 pad 1: /IO25 -> /IO14
- RN3 pad 2: /IO32 -> (no net)
- RN3 pad 3: (no net) -> /IO27
- RN3 pad 4: (no net) -> /IO26
- RN3 pad 5: (no net) -> Net-(RN3-Pad5)
- RN3 pad 6: (no net) -> Net-(RN3-Pad6)
- RN3 pad 7: Net-(RN3-Pad7) -> (no net)
- RN5 pad 1: GND -> /IO25
- RN5 pad 2: GND -> /IO32
- RN5 pad 5: Net-(D12-Pad1) -> Net-(D8-Pad1)
- RN5 pad 6: Net-(D11-Pad1) -> Net-(D7-Pad1)
- RN5 pad 7: Net-(D10-Pad1) -> Net-(RN5-Pad7)
- RN5 pad 8: Net-(D9-Pad1) -> Net-(RN5-Pad8)
- RN6 pad 5: Net-(RN6-Pad5) -> Net-(D12-Pad1)
- RN6 pad 6: Net-(RN6-Pad6) -> Net-(D11-Pad1)
- RN6 pad 7: Net-(D14-Pad1) -> Net-(D10-Pad1)
- RN6 pad 8: Net-(D13-Pad1) -> Net-(D9-Pad1)
- TP1 pad 1: +5V -> Net-(TP1-Pad1)
- U1 pad 13: Net-(U1-Pad13) -> /IO14
- U1 pad 23: Net-(U1-Pad23) -> /IO15
- U1 pad 27: /IO16 -> Net-(U1-Pad27)
- U1 pad 28: /IO17 -> Net-(U1-Pad28)
- U1 pad 29: Net-(U1-Pad29) -> Net-(TP1-Pad1)
- U10 pad 2: Net-(RN2-Pad5) -> Net-(RN5-Pad8)
- U10 pad 7: Net-(J5-Pad6) -> Net-(J5-Pad4)
- U11 pad 2: Net-(RN3-Pad8) -> Net-(RN5-Pad7)
- U11 pad 7: Net-(J5-Pad4) -> Net-(J5-Pad2)
- U2 pad 2: +3V3 -> Net-(RN1-Pad8)
- U2 pad 3: +5V -> GND
- U3 pad 2: Net-(RN1-Pad8) -> Net-(RN1-Pad7)
- U3 pad 7: Net-(J4-Pad10) -> Net-(J4-Pad8)
- U4 pad 2: Net-(RN1-Pad7) -> Net-(RN1-Pad6)
- U4 pad 7: Net-(J4-Pad8) -> Net-(J4-Pad6)
- U5 pad 2: Net-(RN1-Pad6) -> Net-(RN2-Pad7)
- U5 pad 7: Net-(J4-Pad6) -> Net-(J4-Pad4)
- U6 pad 2: Net-(RN1-Pad5) -> Net-(RN2-Pad6)
- U6 pad 7: Net-(J4-Pad4) -> Net-(J4-Pad2)
- U7 pad 2: Net-(RN2-Pad8) -> Net-(RN3-Pad8)
- U7 pad 7: Net-(J4-Pad2) -> Net-(J5-Pad10)
- U8 pad 2: Net-(RN2-Pad7) -> Net-(RN3-Pad6)
- U8 pad 7: Net-(J5-Pad10) -> Net-(J5-Pad8)
- U9 pad 2: Net-(RN2-Pad6) -> Net-(RN3-Pad5)
- U9 pad 7: Net-(J5-Pad8) -> Net-(J5-Pad6)
Routing:
- net GND: track 242.1 -> 154.7 mm, vias 98 -> 87
- net /Relay/F2_LIVE: track 263.0 -> 331.0 mm
- net Net-(TP3-Pad1): track 0.00 -> 64.6 mm, vias 0 -> 2
- net Net-(TP4-Pad1): track 0.00 -> 64.2 mm, vias 0 -> 2
- net Net-(RN1-Pad5): track 55.9 -> 0.00 mm
- net Net-(RN2-Pad8): track 52.3 -> 0.00 mm
- net Net-(TP2-Pad1): track 0.00 -> 51.5 mm, vias 0 -> 2
- net /NEUTRAL: track 313.5 -> 264.9 mm
- net +5V: track 40.8 -> 0.00 mm
- net /IO14: track 0.00 -> 35.6 mm
- net Net-(RN3-Pad8): track 11.5 -> 46.0 mm
- net Net-(RN3-Pad6): track 0.00 -> 34.0 mm
- net Net-(TP1-Pad1): track 0.00 -> 33.9 mm, vias 0 -> 2
- net Net-(RN2-Pad7): track 39.8 -> 66.3 mm
- net Net-(RN2-Pad6): track 28.4 -> 53.9 mm
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- removed copper zone on F.Cu, net +5V
Other:
- outline, holes or cut-outs redrawn
- board text added: "4921"
- board text added: "I2C"
- board text added: "IO12"
- board text added: "IO34"
- board text added: "IO35"
- board text added: "IO5"
- board text added: "WARNING! High Voltage present even when triacs are turned off!"
- board text added: "revC"
- board text removed: "5V"
- board text removed: "Warning: revA has PS1 footprint mirrored!"

Commit message: Release revE First Edition
Parts:
- removed C16: 10nF, Capacitor_THT:C_Rect_L10.3mm_W5.0mm_P7.50mm_MKS4
- removed the C3 at (113.5, 80.5)
- removed the C7 at (105.8, 101.8)
- removed the H3 at (138.8, 78.0)
- removed the H5 at (179.8, 78.0)
- removed J2: i2C, Connector_PinHeader_2.54mm:PinHeader_1x04_P2.54mm_Vertical
- removed the J6 at (56.0, 36.5)
- removed R13, R15, R16, R17, R18: 47R, Resistor_THT:R_Axial_DIN0309_L9.0mm_D3.2mm_P5.08mm_Vertical
- removed the R2 at (62.0, 85.0)
- removed REF**: Symbol_HighVoltage_Type2_CopperTop_VerySmall, Symbol:Symbol_HighVoltage_Type2_CopperTop_VerySmall
- removed TP1: IO5, TestPoint:TestPoint_Pad_D1.5mm
- removed TP2: IO12, TestPoint:TestPoint_Pad_D1.5mm
- removed TP3: IO34, TestPoint:TestPoint_Pad_D1.5mm
- removed TP4: IO35, TestPoint:TestPoint_Pad_D1.5mm
- added C19: 220uF, Capacitor_SMD:CP_Elec_6.3x7.7, F.Cu at (121.2, 80.5)
- added C5: 0.1uF, Capacitor_SMD:C_0402_1005Metric, F.Cu at (124.0, 104.8)
- added C9: 10nF, Capacitor_THT:C_Rect_L10.0mm_W4.0mm_P7.50mm_MKS4, F.Cu at (102.5, 46.2)
- added J7: AC IN, Voltlog:TerminalBlock_1x02_P5.00mm_Horizontal, F.Cu at (53.8, 36.0)
- added J8: Expansion, Voltlog:JST_SH_SM10B-SRSS-TB_1x10-1MP_P1.00mm_Horizontal, F.Cu at (127.0, 108.0)
- added JP1: NEUTRAL, Resistor_SMD:R_2512_6332Metric, F.Cu at (61.2, 38.2)
- added JP2: LIVE, Resistor_SMD:R_2512_6332Metric, F.Cu at (50.8, 45.5)
- added N2: LightPipe, Voltlog:1272.1020, F.Cu at (155.5, 79.0)
- added Q1: AO3400A, Package_TO_SOT_SMD:SOT-23, F.Cu at (128.2, 73.2)
- added R9: 47R, Resistor_SMD:R_1206_3216Metric, F.Cu at (136.8, 47.5)
- added RN1: 4K7, Resistor_SMD:R_Array_Convex_4x0603, F.Cu at (132.5, 98.8)
- added RN2: 100R, Resistor_SMD:R_Array_Convex_4x0603, F.Cu at (132.5, 91.8)
- added kibuzzard-654A0597: G***, kibuzzard-654A0597, F.Cu at (97.2, 104.2)
- added kibuzzard-654A05B0: G***, kibuzzard-654A05B0, F.Cu at (100.2, 104.2)
- added kibuzzard-654A05C3: G***, kibuzzard-654A05C3, F.Cu at (109.8, 101.8)
- added kibuzzard-654A05E9: G***, kibuzzard-654A05E9, F.Cu at (142.2, 102.8)
- added kibuzzard-654A0611: G***, kibuzzard-654A0611, F.Cu at (127.2, 102.8)
- C10, C11, C12, C13, C14, C15: footprint Capacitor_THT:C_Rect_L10.3mm_W5.0mm_P7.50mm_MKS4 -> Capacitor_THT:C_Rect_L10.0mm_W4.0mm_P7.50mm_MKS4
- C17: value 10nF -> 0.1uF; footprint Capacitor_THT:C_Rect_L10.3mm_W5.0mm_P7.50mm_MKS4 -> Capacitor_THT:C_Rect_L13.0mm_W5.0mm_P10.00mm_FKS3_FKP3_MKS4
- C18: value 10nF -> 0.1uF; footprint Capacitor_THT:C_Rect_L10.3mm_W5.0mm_P7.50mm_MKS4 -> Capacitor_SMD:C_0402_1005Metric
- C2: footprint Capacitor_THT:C_Rect_L13.0mm_W5.0mm_P10.00mm_FKS3_FKP3_MKS4 -> Capacitor_SMD:C_0402_1005Metric
- C3: renamed from C1; footprint Capacitor_SMD:C_0603_1608Metric -> Capacitor_SMD:C_0402_1005Metric
- C4: value 220uF -> 0.1uF; footprint Capacitor_SMD:CP_Elec_8x10.5 -> Capacitor_SMD:C_0402_1005Metric
- C6, C8: value 0.1uF -> 10nF; footprint Capacitor_SMD:C_0603_1608Metric -> Capacitor_THT:C_Rect_L10.0mm_W4.0mm_P7.50mm_MKS4
- C7: renamed from C9; footprint Capacitor_THT:C_Rect_L10.3mm_W5.0mm_P7.50mm_MKS4 -> Capacitor_THT:C_Rect_L10.0mm_W4.0mm_P7.50mm_MKS4
- D2: value LED -> USER
- F1: value 0.5A 250VAC -> 1A 250VAC
- F2: value 1A 250VAC -> 0.5A 250VAC; footprint Fuse:Fuseholder_Cylinder-5x20mm_Stelvio-Kontek_PTF78_Horizontal_Open -> Voltlog:Fuse_2410
- FL1: value EMI_Filter_LL -> 15mH; footprint voltlog:UU9_choke -> Voltlog:PSSQAQ1212-153M
- J1: value 1Wire -> VoltLink_target; footprint Connector_PinHeader_2.54mm:PinHeader_1x03_P2.54mm_Vertical -> Voltlog:VoltLink-vertical
- J3: value VoltLink_target -> VALVE IN; footprint Voltlog:VoltLink -> Voltlog:TerminalBlock_1x02_P5.00mm_Horizontal
- J5: renamed from J4; footprint TerminalBlock_RND:TerminalBlock_RND_205-00020_1x10_P5.00mm_Horizontal -> Voltlog:TerminalBlock_1x10_P5.00mm_Horizontal
- J6: renamed from J5; footprint TerminalBlock_RND:TerminalBlock_RND_205-00020_1x10_P5.00mm_Horizontal -> Voltlog:TerminalBlock_1x10_P5.00mm_Horizontal
- PS1: footprint Converter_ACDC:Converter_ACDC_HiLink_HLK-PMxx -> Voltlog:Converter_ACDC_HiLink_HLK-PMxx
- R1: footprint Resistor_SMD:R_0603_1608Metric -> Resistor_SMD:R_0402_1005Metric
- R10, R11, R12: footprint Resistor_THT:R_Axial_DIN0309_L9.0mm_D3.2mm_P5.08mm_Vertical -> Resistor_SMD:R_1206_3216Metric
- R14: value 47R -> 1M; footprint Resistor_THT:R_Axial_DIN0309_L9.0mm_D3.2mm_P5.08mm_Vertical -> Resistor_SMD:R_2010_5025Metric
- R2: renamed from R9; footprint Resistor_THT:R_Axial_DIN0309_L9.0mm_D3.2mm_P5.08mm_Vertical -> Resistor_SMD:R_1206_3216Metric
- R3, R4, R7: value 4K7 -> 47R; footprint Resistor_SMD:R_0603_1608Metric -> Resistor_SMD:R_1206_3216Metric
- R6: value 330R -> 47R; footprint Resistor_SMD:R_0603_1608Metric -> Resistor_SMD:R_1206_3216Metric
- R8: value 100R -> 47R; footprint Resistor_SMD:R_0603_1608Metric -> Resistor_SMD:R_1206_3216Metric
- RV1: footprint Varistor:RV_Disc_D12mm_W5.8mm_P7.5mm -> Varistor:RV_Disc_D12mm_W6.1mm_P7.5mm
- SW1: footprint Button_Switch_THT:SW_Tactile_SKHH_Angled -> Voltlog:TS1045AD
- U10, U11, U2, U3, U4, U5, U6, U7, U8, U9: footprint voltlog:SOIC-7 -> Voltlog:SOIC-7
- V1: footprint voltlog:voltlog_mask_5mm -> Voltlog:voltlog_silk_5mm
- moved C6 115.2 mm to (76.5, 46.2)
- moved C17 110.2 mm to (54.8, 79.5), turned to -90 degrees
- moved C2 104.5 mm to (177.0, 102.4), turned to 90 degrees
- moved J3 99.2 mm to (73.8, 36.0)
- moved R14 82.1 mm to (49.8, 84.0), turned to -90 degrees
- moved R3 80.2 mm to (71.8, 47.5), turned to 180 degrees
- moved R10 79.0 mm to (149.8, 47.5), turned to 180 degrees
- moved R11 79.0 mm to (162.8, 47.5), turned to 180 degrees
- moved R12 77.3 mm to (174.0, 47.5), turned to 90 degrees
- moved V1 72.6 mm to (144.2, 88.0)
- moved R4 70.2 mm to (84.8, 47.5), turned to 180 degrees
- moved C18 65.8 mm to (115.2, 80.7), turned to -90 degrees
- moved R8 63.0 mm to (123.8, 47.5), turned to 180 degrees
- moved C8 62.1 mm to (89.5, 46.2)
- moved R6 58.5 mm to (97.8, 47.5), turned to 180 degrees
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- renumbered C5 to C1, H1 to H3, H2 to H4, H4 to H5, RN1 to RN3, RN2 to RN5, RN5 to RN6, RN6 to RN7, RN3 to RN8
Connections:
- C10 pad 2: /Relay/F2_LIVE -> /Relay/TRIAC_FUSED_LIVE
- C11 pad 2: /Relay/F2_LIVE -> /Relay/TRIAC_FUSED_LIVE
- C12 pad 2: /Relay/F2_LIVE -> /Relay/TRIAC_FUSED_LIVE
- C13 pad 2: /Relay/F2_LIVE -> /Relay/TRIAC_FUSED_LIVE
- C14 pad 2: /Relay/F2_LIVE -> /Relay/TRIAC_FUSED_LIVE
- C15 pad 2: /Relay/F2_LIVE -> /Relay/TRIAC_FUSED_LIVE
- C17 pad 1: Net-(C17-Pad1) -> /ACDC Converter/240V_FUSED_LIVE
- C17 pad 2: /Relay/F2_LIVE -> /240V_NEUTRAL
- C18 pad 1: Net-(C18-Pad1) -> GND
- C18 pad 2: /Relay/F2_LIVE -> +3V3
- C2 pad 1: /F1_LIVE -> GND
- C2 pad 2: /NEUTRAL -> +3V3
- C4 pad 1: +3V3 -> /IO34
- C6 pad 1: +3V3 -> Net-(C6-Pad1)
- C6 pad 2: GND -> /Relay/TRIAC_FUSED_LIVE
- C7 pad 2: /Relay/F2_LIVE -> /Relay/TRIAC_FUSED_LIVE
- C8 pad 1: GND -> Net-(C8-Pad1)
- C8 pad 2: +3V3 -> /Relay/TRIAC_FUSED_LIVE
- D1 pad 2: Net-(D1-Pad2) -> Net-(D1-A)
- D2 pad 2: Net-(D2-Pad2) -> Net-(D2-A)
- D3 pad 1: Net-(D3-Pad1) -> Net-(D3-K)
- D4 pad 1: Net-(D4-Pad1) -> Net-(D4-K)
- D5 pad 1: Net-(D5-Pad1) -> Net-(D5-K)
- D6 pad 1: Net-(D6-Pad1) -> Net-(D6-K)
- F1 pad 1: /F1_LIVE -> /LIVE
- F1 pad 2: /Relay/LIVE -> /Relay/TRIAC_FUSED_LIVE
- F2 pad 1: /Relay/LIVE -> /ACDC Converter/240V_FUSED_LIVE
- F2 pad 2: /Relay/F2_LIVE -> /240V_LIVE
- FL1 pad 1: /NEUTRAL -> /240V_NEUTRAL
- FL1 pad 2: Net-(FL1-Pad2) -> /ACDC Converter/240V_FUSED_LIVE
- FL1 pad 3: /F1_LIVE -> Net-(PS1-AC/L)
- FL1 pad 4: Net-(FL1-Pad4) -> Net-(PS1-AC/N)
- J1 pad 1: /IO4 -> +3V3
- J1 pad 2: +3V3 -> GND
- J1 pad 3: GND -> /TXD
- J3 pad 1: +3V3 -> /NEUTRAL
- J3 pad 2: GND -> /LIVE
- J5 pad 2: Net-(J4-Pad2) -> Net-(J5-Pin_2)
- J5 pad 4: Net-(J4-Pad4) -> Net-(J5-Pin_4)
- J5 pad 6: Net-(J4-Pad6) -> Net-(J5-Pin_6)
- J5 pad 8: Net-(J4-Pad8) -> Net-(J5-Pin_8)
- J6 pad 10: Net-(J5-Pad10) -> Net-(J6-Pin_10)
- J6 pad 2: Net-(J5-Pad2) -> Net-(J6-Pin_2)
- J6 pad 4: Net-(J5-Pad4) -> Net-(J6-Pin_4)
- J6 pad 6: Net-(J5-Pad6) -> Net-(J6-Pin_6)
- PS1 pad 1: Net-(FL1-Pad4) -> Net-(PS1-AC/L)
- PS1 pad 2: Net-(FL1-Pad2) -> Net-(PS1-AC/N)
- R10 pad 1: Net-(C10-Pad1) -> Net-(C13-Pad1)
- R10 pad 2: Net-(J4-Pad8) -> Net-(J6-Pin_6)
- R11 pad 1: Net-(C11-Pad1) -> Net-(C14-Pad1)
- R11 pad 2: Net-(J4-Pad6) -> Net-(J6-Pin_4)
- R12 pad 1: Net-(C12-Pad1) -> Net-(C15-Pad1)
- R12 pad 2: Net-(J4-Pad4) -> Net-(J6-Pin_2)
- R14 pad 1: Net-(C14-Pad1) -> /ACDC Converter/240V_FUSED_LIVE
- R14 pad 2: Net-(J5-Pad10) -> /240V_NEUTRAL
- R3 pad 1: /SDA -> Net-(C6-Pad1)
- R3 pad 2: +3V3 -> Net-(J5-Pin_8)
- R4 pad 1: /SCL -> Net-(C8-Pad1)
- R4 pad 2: +3V3 -> Net-(J5-Pin_6)
- R5 pad 1: /IO33 -> GND
- R5 pad 2: +3V3 -> /IO16
- R6 pad 1: Net-(D1-Pad2) -> Net-(C9-Pad1)
- R6 pad 2: +3V3 -> Net-(J5-Pin_4)
- R7 pad 1: +3V3 -> Net-(C10-Pad1)
- R7 pad 2: /IO4 -> Net-(J5-Pin_2)
- R8 pad 1: Net-(D2-Pad2) -> Net-(C11-Pad1)
- R8 pad 2: /IO2 -> Net-(J6-Pin_10)
- RN4 pad 1: GND -> Net-(D3-K)
- RN4 pad 2: GND -> Net-(D4-K)
- RN4 pad 3: GND -> Net-(D5-K)
- RN4 pad 4: GND -> Net-(D6-K)
- RN4 pad 5: Net-(D6-Pad1) -> Net-(Q1-D)
- RN4 pad 6: Net-(D5-Pad1) -> Net-(Q1-D)
- RN4 pad 7: Net-(D4-Pad1) -> Net-(Q1-D)
- RN4 pad 8: Net-(D3-Pad1) -> Net-(Q1-D)
- RN6 pad 3: GND -> Net-(Q1-D)
- RN6 pad 4: GND -> Net-(Q1-D)
- RN7 pad 1: GND -> Net-(Q1-D)
- RN7 pad 2: GND -> Net-(Q1-D)
- RN7 pad 3: GND -> Net-(Q1-D)
- RN7 pad 4: GND -> Net-(Q1-D)
- RV1 pad 1: /F1_LIVE -> /ACDC Converter/240V_FUSED_LIVE
- RV1 pad 2: /NEUTRAL -> /240V_NEUTRAL
- SW1 pad 1: /IO33 -> /IO34
- U1 pad 14: Net-(TP2-Pad1) -> /IO12
- U1 pad 17: Net-(U1-Pad17) -> unconnected-(U1-SHD/SD2-Pad17)
- U1 pad 18: Net-(U1-Pad18) -> unconnected-(U1-SWP/SD3-Pad18)
- U1 pad 19: Net-(U1-Pad19) -> unconnected-(U1-SCS/CMD-Pad19)
- U1 pad 20: Net-(U1-Pad20) -> unconnected-(U1-SCK/CLK-Pad20)
- U1 pad 21: Net-(U1-Pad21) -> unconnected-(U1-SDO/SD0-Pad21)
- U1 pad 22: Net-(U1-Pad22) -> unconnected-(U1-SDI/SD1-Pad22)
- U1 pad 27: Net-(U1-Pad27) -> /IO16
- U1 pad 28: Net-(U1-Pad28) -> unconnected-(U1-IO17-Pad28)
- U1 pad 29: Net-(TP1-Pad1) -> /IO5
- U1 pad 32: Net-(U1-Pad32) -> unconnected-(U1-NC-Pad32)
- U1 pad 4: Net-(U1-Pad4) -> unconnected-(U1-SENSOR_VP-Pad4)
- U1 pad 5: Net-(U1-Pad5) -> unconnected-(U1-SENSOR_VN-Pad5)
- U1 pad 6: Net-(TP3-Pad1) -> /IO34
- U1 pad 7: Net-(TP4-Pad1) -> unconnected-(U1-IO35-Pad7)
- U10 pad 5: /Relay/F2_LIVE -> /Relay/TRIAC_FUSED_LIVE
- U10 pad 6: /Relay/F2_LIVE -> /Relay/TRIAC_FUSED_LIVE
- U10 pad 7: Net-(J5-Pad4) -> Net-(J6-Pin_4)
- U11 pad 5: /Relay/F2_LIVE -> /Relay/TRIAC_FUSED_LIVE
- U11 pad 6: /Relay/F2_LIVE -> /Relay/TRIAC_FUSED_LIVE
- U11 pad 7: Net-(J5-Pad2) -> Net-(J6-Pin_2)
- U2 pad 5: /Relay/F2_LIVE -> /Relay/TRIAC_FUSED_LIVE
- U2 pad 6: /Relay/F2_LIVE -> /Relay/TRIAC_FUSED_LIVE
- U3 pad 5: /Relay/F2_LIVE -> /Relay/TRIAC_FUSED_LIVE
- U3 pad 6: /Relay/F2_LIVE -> /Relay/TRIAC_FUSED_LIVE
- U3 pad 7: Net-(J4-Pad8) -> Net-(J5-Pin_8)
- U4 pad 5: /Relay/F2_LIVE -> /Relay/TRIAC_FUSED_LIVE
- U4 pad 6: /Relay/F2_LIVE -> /Relay/TRIAC_FUSED_LIVE
- U4 pad 7: Net-(J4-Pad6) -> Net-(J5-Pin_6)
- U5 pad 5: /Relay/F2_LIVE -> /Relay/TRIAC_FUSED_LIVE
- U5 pad 6: /Relay/F2_LIVE -> /Relay/TRIAC_FUSED_LIVE
- U5 pad 7: Net-(J4-Pad4) -> Net-(J5-Pin_4)
- U6 pad 5: /Relay/F2_LIVE -> /Relay/TRIAC_FUSED_LIVE
- U6 pad 6: /Relay/F2_LIVE -> /Relay/TRIAC_FUSED_LIVE
- U6 pad 7: Net-(J4-Pad2) -> Net-(J5-Pin_2)
- U7 pad 5: /Relay/F2_LIVE -> /Relay/TRIAC_FUSED_LIVE
- U7 pad 6: /Relay/F2_LIVE -> /Relay/TRIAC_FUSED_LIVE
- U7 pad 7: Net-(J5-Pad10) -> Net-(J6-Pin_10)
- U8 pad 5: /Relay/F2_LIVE -> /Relay/TRIAC_FUSED_LIVE
- U8 pad 6: /Relay/F2_LIVE -> /Relay/TRIAC_FUSED_LIVE
- U9 pad 5: /Relay/F2_LIVE -> /Relay/TRIAC_FUSED_LIVE
- U9 pad 6: /Relay/F2_LIVE -> /Relay/TRIAC_FUSED_LIVE
- U9 pad 7: Net-(J5-Pad6) -> Net-(J6-Pin_6)
Routing:
- net /Relay/F2_LIVE: track 331.0 -> 0.00 mm
- net /Relay/TRIAC_FUSED_LIVE: track 0.00 -> 292.2 mm
- net /NEUTRAL: track 264.9 -> 176.2 mm
- net /IO34: track 0.00 -> 88.3 mm, vias 0 -> 4
- net /240V_NEUTRAL: track 0.00 -> 87.8 mm
- net /IO12: track 0.00 -> 65.8 mm
- net Net-(TP3-Pad1): track 64.6 -> 0.00 mm, vias 2 -> 0
- net Net-(TP4-Pad1): track 64.2 -> 0.00 mm, vias 2 -> 0
- net Net-(Q1-D): track 0.00 -> 53.3 mm
- net /F1_LIVE: track 53.1 -> 0.00 mm
- net Net-(TP2-Pad1): track 51.5 -> 0.00 mm, vias 2 -> 0
- net /Relay/LIVE: track 45.4 -> 0.00 mm
- net /IO2: track 76.0 -> 31.7 mm, vias 4 -> 0
- net /IO16: track 0.00 -> 43.9 mm, vias 0 -> 2
- net Net-(D1-A): track 0.00 -> 42.6 mm
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- added copper zone on B.Cu, net /LIVE
- added copper zone on F.Cu, net /LIVE
- removed copper zone on F.Cu, net (none)
Other:
- outline, holes or cut-outs redrawn
- net class Default removed
- net class Mains removed
- board text added: "10ch Valve Actuator 24-240VAC 0.3A/ch"
- board text added: "4523"
- board text added: "AC MAINS INPUT 110-240VAC"
- board text added: "BOARD PWR INPUT 110-240VAC"
- board text added: "CH1 - IO23"
- board text added: "CH10 - IO32"
- board text added: "CH2 - IO19"
- board text added: "CH3 - IO18"
- board text added: "CH4 - IO15"
- board text added: "CH5 - IO13"
- board text added: "CH6 - IO14"
- board text added: "CH7 - IO27"
- board text added: "CH8 - IO26"
- board text added: "CH9 - IO25"
- board text added: "DO NOT CONNECT BOTH AT THE SAME TIME UNLESS JP1-JP2 ARE DNP!"
- board text added: "F1=1.0A F2=0.5A"
- board text added: "FIRST EDITION"
- board text added: "IMPORTANT WIRING INFO IF VALVE AND BOARD SHARE SAME AC VOLTAGE BETWEEN 110-240VAC JP1, JP2 ARE INSTALLED AND ONLY J3 INPUT CONNECTOR SHOULD BE USED. IF VALVE AND BOARD USE DIFFERENT VOLTAGES, JP1-JP2 ARE REMOVED, J7 IS USED TO POWER BOARD WITH 110-240VAC, J3 IS USED TO POWER VALVES WITH 24-240VAC."
- board text added: "IO33"
- board text added: "SWITCH IO34"
- board text added: "VALVE PWR"
- board text added: "VALVE PWR INPUT 24-240VAC"
- board text added: "WARNING! High Voltage present even when triacs are turned off due to leakage!"
- board text added: "Warning! High Voltage!"
- board text added: "revD"
- board text removed: "0.25A"
- board text removed: "10ch Valve Actuator 240VAC 0.3A/ch"
- board text removed: "1A"
- board text removed: "1WIRE"
- board text removed: "4921"
- board text removed: "AC MAINS INPUT"
- board text removed: "F1=0.25A F2=1A"
- board text removed: "I2C"
- board text removed: "IO2"
- board text removed: "IO35"
- board text removed: "VOLTLINK"
- board text removed: "WARNING! High Voltage present even when triacs are turned off!"
- board text removed: "Warning! High Voltage! 110-240VAC"
- board text removed: "revC"
