File: relay.sch (KiCad schematic (older format))
At the start: 50 parts, among them J4 OUTPUT, J5 OUTPUT, J6 AC IN, U10 BC3223, U11 BC3223, U12 BC3223, U3 BC3223, U4 BC3223, U5 BC3223, U6 BC3223, U7 BC3223, U8 BC3223, U9 BC3223

Commit message: revB release
Parts:
- J4, J5: footprint Voltlog:KF235-5.0-10P -> TerminalBlock_RND:TerminalBlock_RND_205-00020_1x10_P5.00mm_Horizontal
- J6: footprint Voltlog:KF235-5.0-2P -> TerminalBlock_RND:TerminalBlock_RND_205-00012_1x02_P5.00mm_Horizontal
- R10, R11, R12, R13, R14, R15, R16, R17, R18, R9: footprint Resistor_THT:R_Axial_DIN0207_L6.3mm_D2.5mm_P10.16mm_Horizontal -> Resistor_THT:R_Axial_DIN0309_L9.0mm_D3.2mm_P5.08mm_Vertical
- RN1, RN2, RN3: value 100R -> 75R
- U10: renamed from U11; value BC3223 -> BC2213A; footprint voltlog:DIP-7_W7.62mm -> voltlog:SOIC-7
- U11: renamed from U12; value BC3223 -> BC2213A; footprint voltlog:DIP-7_W7.62mm -> voltlog:SOIC-7
- U2: renamed from U3; value BC3223 -> BC2213A; footprint voltlog:DIP-7_W7.62mm -> voltlog:SOIC-7
- U3: renamed from U4; value BC3223 -> BC2213A; footprint voltlog:DIP-7_W7.62mm -> voltlog:SOIC-7
- U4: renamed from U5; value BC3223 -> BC2213A; footprint voltlog:DIP-7_W7.62mm -> voltlog:SOIC-7
- U5: renamed from U6; value BC3223 -> BC2213A; footprint voltlog:DIP-7_W7.62mm -> voltlog:SOIC-7
- U6: renamed from U7; value BC3223 -> BC2213A; footprint voltlog:DIP-7_W7.62mm -> voltlog:SOIC-7
- U7: renamed from U8; value BC3223 -> BC2213A; footprint voltlog:DIP-7_W7.62mm -> voltlog:SOIC-7
- U8: renamed from U9; value BC3223 -> BC2213A; footprint voltlog:DIP-7_W7.62mm -> voltlog:SOIC-7
- U9: renamed from U10; value BC3223 -> BC2213A; footprint voltlog:DIP-7_W7.62mm -> voltlog:SOIC-7
- renumbered C11 to C10, C12 to C11, C13 to C12, C14 to C13, C15 to C14, C16 to C15, C17 to C16, C18 to C17, C19 to C18, C10 to C9, D12 to D10, D13 to D11, D14 to D12, D5 to D3, D6 to D4, D7 to D5, D8 to D6, D9 to D7, D10 to D8, D11 to D9
Connections:
- net at J4.10 (Pin_10), U2.7: now also R9.2; no longer R9.1
- net at J4.2 (Pin_2), U6.7: now also R13.2; no longer R13.1
- net at J4.4 (Pin_4), U5.7: now also R12.2; no longer R12.1
- net at J4.6 (Pin_6), U4.7: now also R11.2; no longer R11.1
- net at J4.8 (Pin_8), U3.7: now also R10.2; no longer R10.1
- net at J5.10 (Pin_10), U7.7: now also R14.2; no longer R14.1
- net at J5.2 (Pin_2), U11.7: now also R18.2; no longer R18.1
- net at J5.4 (Pin_4), U10.7: now also R17.2; no longer R17.1
- net at J5.6 (Pin_6), U9.7: now also R16.2; no longer R16.1
- net at J5.8 (Pin_8), U8.7: now also R15.2; no longer R15.1
- net at C9.1: now also R9.1; no longer R9.2
- net at C10.1: now also R10.1; no longer R10.2
- net at C11.1: now also R11.1; no longer R11.2
- net at C12.1: now also R12.1; no longer R12.2
- net at C13.1: now also R13.1; no longer R13.2
- net at C14.1: now also R14.1; no longer R14.2
- net at C15.1: now also R15.1; no longer R15.2
- net at C16.1: now also R16.1; no longer R16.2
- net at C17.1: now also R17.1; no longer R17.2
- net at C18.1: now also R18.1; no longer R18.2
Other:
- note added: "WARNING: TRIACS by their nature have structural leakage current in the off state, \nwhich is why a small amount of current flows through the load. The snubber circuit \nalso contributes to that effect and ads it's own leakage current so we end up with \naproximately 700uA at each output. When a load like a resistive thermostat valve is \nconnected, the voltage at the output will drop to about 1-2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"
