File: relay.sch (KiCad schematic (older format))
At the start: 50 parts, among them J4 OUTPUT, J5 OUTPUT, J6 AC IN, U10 BC3223, U11 BC3223, U12 BC3223, U3 BC3223, U4 BC3223, U5 BC3223, U6 BC3223, U7 BC3223, U8 BC3223, U9 BC3223

Commit message: RevC initial release
Parts:
- removed unit 4 of RN1
- removed unit 1 of RN2
- removed unit 2 of RN3
- removed RN5: 100R, Resistor_SMD:R_Array_Convex_4x0603, symbol Device:R_Pack04
- added unit 4 of RN3
- added unit 3 of RN3
- added unit 3 of RN5
- added unit 2 of RN5
- added unit 1 of RN5
- J4, J5: footprint Voltlog:KF235-5.0-10P -> TerminalBlock_RND:TerminalBlock_RND_205-00020_1x10_P5.00mm_Horizontal
- J6: footprint Voltlog:KF235-5.0-2P -> TerminalBlock_RND:TerminalBlock_RND_205-00012_1x02_P5.00mm_Horizontal
- R10, R11, R12, R13, R14, R15, R16, R17, R18, R9: footprint Resistor_THT:R_Axial_DIN0207_L6.3mm_D2.5mm_P10.16mm_Horizontal -> Resistor_THT:R_Axial_DIN0309_L9.0mm_D3.2mm_P5.08mm_Vertical
- U10: renamed from U11; value BC3223 -> BC2213A; footprint voltlog:DIP-7_W7.62mm -> voltlog:SOIC-7
- U11: renamed from U12; value BC3223 -> BC2213A; footprint voltlog:DIP-7_W7.62mm -> voltlog:SOIC-7
- U2: renamed from U3; value BC3223 -> BC2213A; footprint voltlog:DIP-7_W7.62mm -> voltlog:SOIC-7
- U3: renamed from U4; value BC3223 -> BC2213A; footprint voltlog:DIP-7_W7.62mm -> voltlog:SOIC-7
- U4: renamed from U5; value BC3223 -> BC2213A; footprint voltlog:DIP-7_W7.62mm -> voltlog:SOIC-7
- U5: renamed from U6; value BC3223 -> BC2213A; footprint voltlog:DIP-7_W7.62mm -> voltlog:SOIC-7
- U6: renamed from U7; value BC3223 -> BC2213A; footprint voltlog:DIP-7_W7.62mm -> voltlog:SOIC-7
- U7: renamed from U8; value BC3223 -> BC2213A; footprint voltlog:DIP-7_W7.62mm -> voltlog:SOIC-7
- U8: renamed from U9; value BC3223 -> BC2213A; footprint voltlog:DIP-7_W7.62mm -> voltlog:SOIC-7
- U9: renamed from U10; value BC3223 -> BC2213A; footprint voltlog:DIP-7_W7.62mm -> voltlog:SOIC-7
- renumbered C11 to C10, C12 to C11, C13 to C12, C14 to C13, C15 to C14, C16 to C15, C17 to C16, C18 to C17, C19 to C18, C10 to C9, D12 to D10, D13 to D11, D14 to D12, D5 to D3, D6 to D4, D7 to D5, D8 to D6, D9 to D7, D10 to D8, D11 to D9, RN2 to RN5
Connections:
- net CH10: now also RN5.2 (R2.1)
- net CH4: now also RN2.2 (R2.1)
- net CH5: now also RN2.3 (R3.1)
- net CH6: now also RN3.1 (R1.1); no longer RN2.2 (R2.1)
- net CH7: now also RN3.3 (R3.1); no longer RN2.3 (R3.1)
- net CH8: now also RN3.4 (R4.1); no longer RN5.4 (R4.1)
- net CH9: now also RN5.1 (R1.1); no longer RN3.1 (R1.1)
- net GND: now also RN5.4 (R4.1), RN5.3 (R3.1)
- net at J4.10 (Pin_10), U2.7: now also R9.2; no longer R9.1
- net at J4.2 (Pin_2), U6.7: now also R13.2; no longer R13.1
- net at J4.4 (Pin_4), U5.7: now also R12.2; no longer R12.1
- net at J4.6 (Pin_6), U4.7: now also R11.2; no longer R11.1
- net at J4.8 (Pin_8), U3.7: now also R10.2; no longer R10.1
- net at J5.10 (Pin_10), U7.7: now also R14.2; no longer R14.1
- net at J5.2 (Pin_2), U11.7: now also R18.2; no longer R18.1
- net at J5.4 (Pin_4), U10.7: now also R17.2; no longer R17.1
- net at J5.6 (Pin_6), U9.7: now also R16.2; no longer R16.1
- net at J5.8 (Pin_8), U8.7: now also R15.2; no longer R15.1
- net at D7.1 (K): now also RN5.6 (R3.2)
- net at D8.1 (K): now also RN5.5 (R4.2)
- net at D9.1 (K): now also RN6.8 (R1.2)
- net at D10.1 (K): now also RN6.7 (R2.2)
- net at D11.1 (K): now also RN6.6 (R3.2); no longer RN6.8 (R1.2)
- net at D12.1 (K): now also RN6.5 (R4.2); no longer RN6.7 (R2.2)
- net at C9.1: now also R9.1; no longer R9.2
- net at C10.1: now also R10.1; no longer R10.2
- net at C11.1: now also R11.1; no longer R11.2
- net at U5.2: now also RN2.7 (R2.2)
- net at C12.1: now also R12.1; no longer R12.2
- net at U6.2: now also RN2.6 (R3.2)
- net at C13.1: now also R13.1; no longer R13.2
- net at U7.2: now also RN3.8 (R1.2); no longer RN2.7 (R2.2)
- net at C14.1: now also R14.1; no longer R14.2
- net at U8.2: now also RN3.6 (R3.2); no longer RN2.6 (R3.2)
- net at C15.1: now also R15.1; no longer R15.2
- net at U9.2: now also RN3.5 (R4.2); no longer RN5.5 (R4.2)
- net at C16.1: now also R16.1; no longer R16.2
- net at U10.2: now also RN5.8 (R1.2); no longer RN3.8 (R1.2)
- net at C17.1: now also R17.1; no longer R17.2
- net at U11.2: now also RN5.7 (R2.2)
- net at C18.1: now also R18.1; no longer R18.2
Other:
- note added: "WARNING: TRIACS by their nature have structural leakage current in the off state, \nwhich is why a small amount of current flows through the load. The snubber circuit \nalso contributes to that effect and ads it's own leakage current so we end up with \naproximately 700uA at each output. When a load like a resistive thermostat valve is \nconnected, the voltage at the output will drop to about 1-2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"
- moved on the sheet: RN2B, RN2C, RN5D
