File: controller.sch (KiCad schematic (older format))
At the start: 43 parts, among them J1 1Wire, J2 VoltLink_target, J3 i2C, SW1 USER, U1 ESP32-WROOM-32D, U2 AMS1117-3.3

Commit message: RevC initial release
Parts:
- removed C7: 22uF, Capacitor_SMD:C_1206_3216Metric, symbol Device:C
- removed D1: P6SMB6.8CA, Diode_SMD:D_SMB, symbol Diode:SM6T15A
- removed D2: 5V, LED_SMD:LED_0603_1608Metric, symbol Device:LED
- removed PS1: TAS3-5, voltlog:TDPOWER-TAS3-5, symbol voltlog:TAS3-5
- removed R5: 2K, Resistor_SMD:R_0603_1608Metric, symbol Device:R_US
- removed U2: AMS1117-3.3, Package_TO_SOT_SMD:SOT-223-3_TabPin2, symbol Regulator_Linear:AMS1117-3.3
- added FL1: EMI_Filter_LL, voltlog:UU9_choke, symbol Device:EMI_Filter_LL
- added PS1: HLK-PM03, Converter_ACDC:Converter_ACDC_HiLink_HLK-PMxx, symbol Converter_ACDC:HLK-PM03
- added TP2: IO12, TestPoint:TestPoint_Pad_D1.5mm, symbol Connector:TestPoint
- added TP3: IO34, TestPoint:TestPoint_Pad_D1.5mm, symbol Connector:TestPoint
- added TP4: IO35, TestPoint:TestPoint_Pad_D1.5mm, symbol Connector:TestPoint
- added TP5: 3V3, TestPoint:TestPoint_Pad_D1.5mm, symbol Connector:TestPoint
- C4: renamed from C3; value 470uF -> 220uF; footprint Capacitor_SMD:CP_Elec_10x10 -> Capacitor_SMD:CP_Elec_8x10.5; PN (none) -> FZ1C221M-CRF10
- F1: value 0.25A 250VAC -> 0.5A 250VAC; Type (none) -> Slow
- J1: footprint Voltlog:KF235-5.0-3P -> Connector_PinHeader_2.54mm:PinHeader_1x03_P2.54mm_Vertical
- R2: renamed from R19; footprint Resistor_THT:R_Axial_DIN0207_L6.3mm_D2.5mm_P10.16mm_Horizontal -> Resistor_THT:R_Axial_DIN0309_L9.0mm_D3.2mm_P12.70mm_Horizontal
- RV1: value 10D471K -> 10D561K
- SW1: footprint Button_Switch_SMD:SW_SPST_PTS645 -> Button_Switch_THT:SW_Tactile_SKHH_Angled
- TP1: value 5V -> IO5; footprint TestPoint:TestPoint_Pad_D1.0mm -> TestPoint:TestPoint_Pad_D1.5mm
- renumbered C4 to C2, C2 to C3, C8 to C7, C9 to C8, D3 to D1, D4 to D2, J3 to J2, J2 to J3, R2 to R3, R3 to R4, R4 to R5
Connections:
- net +3V3: now also C3.1, C4.1, PS1.4 (+Vout), TP5.1
- net F1_LIVE: now also FL1.3
- net GND: now also PS1.3 (-Vout)
- net NEUTRAL: now also FL1.1
- net IO14: now reaches U1.13 (IO14)
- net at U1.14 (IO12): now also TP2.1
- net IO15: now reaches U1.23 (IO15)
- net at U1.29 (IO5): now also TP1.1
- net at U1.6 (IO34): now also TP3.1
- net at U1.7 (IO35): now also TP4.1
- removed net +5V: C3.1, C4.1, TP1.1
- net IO16: no longer names the net of U1.27 (IO16)
- net IO17: no longer names the net of U1.28 (IO17)
- new net: FL1.4, PS1.1 (AC/L)
- new net: FL1.2, PS1.2 (AC/N)
Other:
- note added: "GPIO 6, 7, 8, 9, 10, 11, 16, 17\nshould be avoided with Tasmota"
- note removed: "Note: starting with Tasmota releases newer than v9.5.0 Tasmota started using IO16, IO17\nto connect to external PSRAM and due to the way Tasmota implements this, it continously\ntries to talk to the external PSRAM, without considering the type of hardware, whether\nit contains any PSRAM or not. As a consequence, IO16, IO17 will show constant SPI traffic so \nIT IS RECOMMENDED YOU FLASH REV.A HW W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"
- moved on the sheet: C2, C3, C4, F1, R2, RV1
